File: ZachEKeyboard.kicad_pcb (KiCad board)
At the start: 2 copper layers, 95.6 x 55.2 mm, 26 parts, among them J1 Conn_01x05_Socket, U1 ProMicro

Commit message: Fixed pinout
Connections:
- U1 pad 10: /COL3 -> /COL2
- U1 pad 11: unconnected-(U1-B4-Pad11) -> /COL3
- U1 pad 4: /ROW0 -> unconnected-(U1-GND-Pad4)
- U1 pad 5: /ROW1 -> /ROW0
- U1 pad 6: /ROW2 -> /ROW1
- U1 pad 7: /COL0 -> /ROW2
- U1 pad 8: /COL1 -> /COL0
- U1 pad 9: /COL2 -> /COL1
Routing:
- net /ROW2: track 111.7 -> 107.8 mm
- net /ROW1: track 95.3 -> 92.5 mm
- net /COL3: track 82.1 -> 84.8 mm
- net /COL2: track 98.8 -> 101.4 mm
- net /COL0: track 134.3 -> 136.8 mm
- net /COL1: track 117.2 -> 119.6 mm
- net /ROW0: track 80.1 -> 79.0 mm
