File: ZachEKeyboard.kicad_sch (KiCad schematic)
At the start: 26 parts, among them J1 Conn_01x05_Socket, U1 ProMicro

Commit message: Fixed pinout
Connections:
- net COL0: now also U1.8 (C6); no longer U1.7 (D4)
- net COL1: now also U1.9 (D7); no longer U1.8 (C6)
- net COL2: now also U1.10 (E6); no longer U1.9 (D7)
- net COL3: now also U1.11 (B4); no longer U1.10 (E6)
- net ROW0: now also U1.5 (D1); no longer U1.4 (GND)
- net ROW1: now also U1.6 (D0); no longer U1.5 (D1)
- net ROW2: now also U1.7 (D4); no longer U1.6 (D0)
Changed lines of the file:
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@@
     (effects (font (size 1.27 1.27)) (justify left bottom))
   )
-  (label "ROW0" (at 120.65 72.39 180) (fields_autoplaced)
-    (effects (font (size 1.27 1.27)) (justify right bottom))
-  )
-  (label "ROW2" (at 120.65 77.47 180) (fields_autoplaced)
+  (label "ROW2" (at 120.65 80.01 180) (fields_autoplaced)
     (effects (font (size 1.27 1.27)) (justify right bottom))
   )
@@
     (effects (font (size 1.27 1.27)) (justify right bottom))
   )
-  (label "COL1" (at 120.65 82.55 180) (fields_autoplaced)
+  (label "COL1" (at 120.65 85.09 180) (fields_autoplaced)
     (effects (font (size 1.27 1.27)) (justify right bottom))
   )
-  (label "COL2" (at 120.65 85.09 180) (fields_autoplaced)
+  (label "COL2" (at 120.65 87.63 180) (fields_autoplaced)
     (effects (font (size 1.27 1.27)) (justify right bottom))
   )
@@
     (effects (font (size 1.27 1.27)) (justify right bottom))
   )
-  (label "COL0" (at 120.65 80.01 180) (fields_autoplaced)
+  (label "COL0" (at 120.65 82.55 180) (fields_autoplaced)
     (effects (font (size 1.27 1.27)) (justify right bottom))
   )
-  (label "ROW1" (at 120.65 74.93 180) (fields_autoplaced)
+  (label "ROW1" (at 120.65 77.47 180) (fields_autoplaced)
     (effects (font (size 1.27 1.27)) (justify right bottom))
   )
@@
     (effects (font (size 1.27 1.27)) (justify left bottom))
   )
-  (label "COL3" (at 120.65 87.63 180) (fields_autoplaced)
+  (label "COL3" (at 120.65 90.17 180) (fields_autoplaced)
     (effects (font (size 1.27 1.27)) (justify right bottom))
   )
+  (label "ROW0" (at 120.65 74.93 180) (fields_autoplaced)
+    (effects (font (size 1.27 1.27)) (justify right bottom))
+  )
